Commit message: Updated urdf for autonav and spawn robot in gz

File: autonav_description/urdf/autonav.xacro (robot description, xacro)
@@ -2,5 +2,6 @@
 <robot name="autonav" xmlns:xacro="http://www.ros.org/wiki/xacro">
 <xacro:include filename="$(find autonav_description)/urdf/materials.xacro" />
-<xacro:include filename="$(find autonav_description)/urdf/autonav_gazebo.xacro" />
+<!-- <xacro:include filename="$(find autonav_description)/urdf/autonav_gazebo.xacro" /> -->
+<xacro:include filename="$(find autonav_description)/urdf/autonav_plugins.xacro" />
 <link name="base_footprint"/>
 <link name="base_link">
@@ -18,13 +19,12 @@
   </visual>
   <collision>
-    <!-- <origin xyz="0 0 0" rpy="0 0 0"/>
+    <origin xyz="0 0 0" rpy="0 0 0"/>
     <geometry>
       <mesh filename="package://autonav_description/meshes/base_link.stl" scale="0.001 0.001 0.001"/>
+    </geometry>
+    <!-- <origin xyz="0.04 0 0.005" rpy="0 0 0"/>
+    <geometry>
+      <box size="0.20 0.18 0.01" />
     </geometry> -->
-    <origin xyz="0.04 0 0.005" rpy="0 0 0"/>
-    <geometry>
-      <!-- <mesh filename="package://cube_description/meshes/base_link.stl" scale="0.001 0.001 0.001"/> -->
-      <box size="0.20 0.18 0.01" />
-    </geometry>
   </collision>
 </link>
@@ -65,5 +65,5 @@
   <inertial>
     <origin xyz="-3.3364538596768883e-08 -0.017500170586145114 1.5158223017064376e-08" rpy="0 0 0"/>
-    <mass value="0.1635143859009559"/>
+    <mass value="1.1635143859009559"/>
     <inertia ixx="8.2e-05" iyy="0.000131" izz="8.2e-05" ixy="-0.0" iyz="-0.0" ixz="-0.0"/>
   </inertial>
@@ -81,9 +81,10 @@
     </geometry>
   </collision>
+  <mu>10.0</mu>
 </link>
 <link name="left_wheel_1">
   <inertial>
     <origin xyz="-1.4750377623972896e-09 0.017500000000000668 2.8030050856775457e-08" rpy="0 0 0"/>
-    <mass value="0.1635143859009559"/>
+    <mass value="1.1635143859009559"/>
     <inertia ixx="8.2e-05" iyy="0.000131" izz="8.2e-05" ixy="0.0" iyz="0.0" ixz="0.0"/>
   </inertial>
@@ -101,4 +102,5 @@
     </geometry>
   </collision>
+  <mu>10.0</mu>
 </link>
 <link name="lidar_1">

File: autonav_description/urdf/autonav_gazebo.xacro (robot description, xacro)
@@ -6,18 +6,4 @@
 <xacro:property name="lidar" value="Gazebo/BlueGlow" />
 <xacro:property name="depth_cam" value="Gazebo/TurquoiseGlow" />
-  <transmission name="wheel_right_transmission">
-    <plugin>transmission_interface/SimpleTransmission</plugin>
-    <actuator name="wheel_right_motor" role="actuator_right"/>
-    <joint name="base2right"    role="joint_right">
-      <mechanical_reduction>1.0</mechanical_reduction>
-    </joint>
-  </transmission>
-  <transmission name="wheel_left_transmission">
-    <plugin>transmission_interface/SimpleTransmission</plugin>
-    <actuator name="wheel_left_motor" role="actuator_left"/>
-    <joint name="base2left"    role="joint_left">
-      <mechanical_reduction>1.0</mechanical_reduction>
-    </joint>
-  </transmission>
   <!-- Wheels -->
   <gazebo reference="left_wheel_1">
@@ -78,147 +64,3 @@
     <maxVel>1.0</maxVel>
   </gazebo>
-  <gazebo>
-    <plugin name="diff_drive_control" filename="libgazebo_ros_diff_drive.so">
-      <!-- Update rate in Hz -->
-      <update_rate>50</update_rate>
-      <!-- wheels -->
-      <left_joint>base2left</left_joint>
-      <right_joint>base2right</right_joint>
-      <!-- kinematics -->
-      <wheel_separation>0.21</wheel_separation>
-      <wheel_diameter>0.08</wheel_diameter>
-      <!-- input -->
-      <command_topic>cmd_vel</command_topic>
-      <!-- output -->
-      <publish_odom>true</publish_odom>
-      <publish_odom_tf>true</publish_odom_tf>
-      <publish_wheel_tf>true</publish_wheel_tf>
-      <odometry_topic>odom</odometry_topic>
-      <odometry_frame>odom</odometry_frame>
-      <robot_base_frame>base_footprint</robot_base_frame>
-    </plugin>
-  </gazebo>
-  <gazebo reference="imu_1">
-    <gravity>true</gravity>
-    <sensor name="imu_1" type="imu">
-      <always_on>true</always_on>
-      <update_rate>30</update_rate>
-      <visualize>true</visualize>
-      <plugin name="my_imu_plugin" filename="libgazebo_ros_imu_sensor.so">
-        <ros>
-          <remapping>~/out:=imu</remapping>
-        </ros>
-        <frame_name>imu_1</frame_name>
-      </plugin>
-    </sensor>
-  </gazebo>
-  <gazebo reference="lidar_1">
-    <sensor type="ray" name="head_hokuyo_sensor">
-      <pose>0 0 0 0 0 0</pose>
-      <visualize>false</visualize>
-      <update_rate>30</update_rate>
-      <ray>
-        <scan>
-          <horizontal>
-            <samples>300</samples>
-            <resolution>1</resolution>
-            <min_angle>-3.14</min_angle>
-            <max_angle>3.14</max_angle>
-          </horizontal>
-        </scan>
-        <range>
-          <min>0.10</min>
-          <max>30.0</max>
-          <resolution>0.01</resolution>
-        </range>
-        <noise>
-          <type>gaussian</type>
-          <!-- Noise parameters based on published spec for Hokuyo laser
-               achieving "+-30mm" accuracy at range < 10m.  A mean of 0.0m and
-               stddev of 0.01m will put 99.7% of samples within 0.03m of the true
-               reading. -->
-          <mean>0.0</mean>
-          <stddev>0.01</stddev>
-        </noise>
-      </ray>
-      <plugin name="my_ray_sensor_plugin" filename="libgazebo_ros_ray_sensor.so">
-        <ros>
-          <!-- Configure namespace and remap to publish to /ray/pointcloud2 -->
-          <remapping>~/out:=scan</remapping>
-        </ros>
-        <!-- Output as a PointCloud2, see above for other types -->
-        <output_type>sensor_msgs/LaserScan</output_type>
-        <!-- Clip intensity values so all are above 100, optional -->
-        <min_intensity>100.0</min_intensity>
-        <!-- Frame id for header of output, defaults to sensor's parent link name -->
-        <frame_name>lidar_1</frame_name>
-      </plugin>
-    </sensor>
-  </gazebo>
-  <gazebo reference="camera_link">
-    <sensor name="camera" type="depth">
-      <pose> 0 0 0 0 0 0</pose>
-      <visualize>true</visualize>
-      <update_rate>60.0</update_rate>
-      <camera name="camera_link">
-        <horizontal_fov>1.047198</horizontal_fov>
-        <image>
-          <width>640</width>
-          <height>480</height>
-          <format>R8G8B8</format>
-        </image>
-        <clip>
-          <near>0.05</near>
-          <far>10</far>
-        </clip>
-      </camera>
-      <plugin name="depth_camera_controller" filename="libgazebo_ros_camera.so">
-        <!-- <ros>
-          <remapping>/camera/camera_info:=/camera/rgb/camera_info</remapping>
-          <remapping>/camera/image_raw:=/camera/rgb/image_rect_color</remapping>
-          <remapping>/camera/depth/image_raw:=/camera/depth_registered/image_raw</remapping>
-        </ros> -->
-        <baseline>0.2</baseline>
-        <alwaysOn>true</alwaysOn>
-        <updateRate>0.0</updateRate>
-        <frame_name>camera_link_1</frame_name>
-        <pointCloudCutoff>0.1</pointCloudCutoff>
-        <pointCloudCutoffMax>10.0</pointCloudCutoffMax>
-        <distortionK1>0</distortionK1>
-        <distortionK2>0</distortionK2>
-        <distortionK3>0</distortionK3>
-        <distortionT1>0</distortionT1>
-        <distortionT2>0</distortionT2>
-        <CxPrime>0</CxPrime>
-        <Cx>0</Cx>
-        <Cy>0</Cy>
-        <focalLength>0</focalLength>
-        <hackBaseline>0</hackBaseline>
-      </plugin>
-      <!-- <plugin name="camera_plugin" filename="libgazebo_ros_camera.so">
-        <baseline>0.2</baseline>
-        <alwaysOn>true</alwaysOn>
-        <updateRate>0.0</updateRate>
-        <cameraName>camera_ir</cameraName>
-        <imageTopicName>/camera/color/image_raw</imageTopicName>
-        <cameraInfoTopicName>/camera/color/camera_info</cameraInfoTopicName>
-        <depthImageTopicName>/camera/depth/image_raw</depthImageTopicName>
-        <depthImageCameraInfoTopicName>/camera/depth/camera_info</depthImageCameraInfoTopicName>
-        <pointCloudTopicName>/camera/depth/points</pointCloudTopicName>
-        <frameName>camera_link</frameName>
-        <pointCloudCutoff>0.5</pointCloudCutoff>
-        <pointCloudCutoffMax>3.0</pointCloudCutoffMax>
-        <distortionK1>0</distortionK1>
-        <distortionK2>0</distortionK2>
-        <distortionK3>0</distortionK3>
-        <distortionT1>0</distortionT1>
-        <distortionT2>0</distortionT2>
-        <CxPrime>0</CxPrime>
-        <Cx>0</Cx>
-        <Cy>0</Cy>
-        <focalLength>0</focalLength>
-        <hackBaseline>0</hackBaseline>
-      </plugin> -->
-    </sensor>
-  </gazebo>
 </robot>

Commit message: Teleop Working

File: autonav_description/urdf/autonav.xacro (robot description, xacro)
@@ -23,9 +23,10 @@
       <mesh filename="package://autonav_description/meshes/base_link.stl" scale="0.001 0.001 0.001"/>
     </geometry>
-    <!-- <origin xyz="0.04 0 0.005" rpy="0 0 0"/>
+    <!-- <origin xyz="0.04 0 0.0055" rpy="0 0 0"/>
     <geometry>
       <box size="0.20 0.18 0.01" />
     </geometry> -->
   </collision>
+  <mu>0.0</mu>
 </link>
 <joint name="footprint2baselink" type="fixed">
@@ -81,5 +82,5 @@
     </geometry>
   </collision>
-  <mu>10.0</mu>
+  <mu>5.0</mu>
 </link>
 <link name="left_wheel_1">
@@ -102,5 +103,5 @@
     </geometry>
   </collision>
-  <mu>10.0</mu>
+  <mu>5.0</mu>
 </link>
 <link name="lidar_1">
@@ -153,5 +154,5 @@
   <parent link="base_link"/>
   <child link="right_wheel_1"/>
-  <axis xyz="-0.0 1.0 0.0"/>
+  <axis xyz="0.0 1.0 0.0"/>
 </joint>
 <joint name="base2left" type="continuous">
@@ -159,5 +160,5 @@
   <parent link="base_link"/>
   <child link="left_wheel_1"/>
-  <axis xyz="0.0 1.0 -0.0"/>
+  <axis xyz="0.0 1.0 0.0"/>
 </joint>
 <joint name="base2lidar" type="fixed">

File: autonav_description/urdf/autonav_plugins.xacro (robot description, xacro)
@@ -2,5 +2,5 @@
 <robot xmlns:xacro="http://www.ros.org/wiki/xacro" name="autonav">
     <gazebo>
-        <plugin filename="ignition-gazebo-sensors-system" name="ignition::gazebo::systems::Sensors">
+        <!-- <plugin filename="ignition-gazebo-sensors-system" name="ignition::gazebo::systems::Sensors">
             <render_engine>ogre2</render_engine>
         </plugin>
@@ -8,17 +8,21 @@
         </plugin>
         <plugin filename="ignition-gazebo-joint-state-publisher-system" name="ignition::gazebo::systems::JointStatePublisher">
-        </plugin>
+        </plugin> -->
         <plugin filename="ignition-gazebo-diff-drive-system" name="ignition::gazebo::systems::DiffDrive">
             <left_joint>base2left</left_joint>
-            <right_joint>base2rigth</right_joint>
-            <wheel_separation>0.21</wheel_separation>
-            <wheel_radius>0.04</wheel_radius>
+            <right_joint>base2right</right_joint>
+            <wheel_separation>1.2</wheel_separation>
+            <wheel_radius>0.1</wheel_radius>
             <odom_publish_frequency>30</odom_publish_frequency>
             <topic>/cmd_vel</topic>
+            <!-- <xacro:if value="${odometry_source == 'encoders'}">
+                <odom_topic>$(arg wheel_odom_topic)</odom_topic>
+                <tf_topic>/tf</tf_topic>
+            </xacro:if> -->
             <frame_id>odom</frame_id>
             <child_frame_id>base_link</child_frame_id>
         </plugin>
     </gazebo>
-    <gazebo>
+    <!-- <gazebo>
         <plugin filename="libignition-gazebo6-odometry-publisher-system"
             name="ignition::gazebo::systems::OdometryPublisher">
@@ -30,6 +34,6 @@
             <odom_publish_frequency>10</odom_publish_frequency>
         </plugin>
-    </gazebo>
-    <gazebo reference="lidar_1">
+    </gazebo> -->
+    <!-- <gazebo reference="lidar_1">
         <sensor name='gpu_lidar' type='gpu_lidar'>
             <topic>scan</topic>
@@ -59,4 +63,4 @@
             <visualize>true</visualize>
         </sensor>
-    </gazebo>
+    </gazebo> -->
 </robot>
